File: pcb/pcb/boneclamp_rB.brd (EAGLE design)
At the start: 160 x 100 mm, 72 parts, among them IC1 24C, U1 AD8032ARZ-REEL7, U2 LT1964ES5-5TRMPBF, U4 TLV70245DBVT, U7 AD7682BCPZ, U8 TPS63700DRCT, U9 ADA4841-2YRZ

Commit message: Added voltage biasing
Parts:
- removed U9: ADA4841-2YRZ, analog-devices-01:SOIC127P600X175-8N
- added C19, C20, C21, C25, C3, C4: (no value), resistor:C025-025X050
- added R17: 6.66k, resistor:0204V
- added R18, R20: 10k, resistor:0204V
- added R19: 6.937k, resistor:0204V
- added R21, R22, R23, R24, R25, R26, R27, R28: (no value), resistor:0204V
- added R29, R38, R43, R44: 0.1k, rcl:R0805
- added R39, R40, R41, R42: 10k, rcl:R0805
- added U10, U11, U3: ADA4841-2YRZ, analog-devices-01:SOIC127P600X175-8N
- added U6: AD713JRZ-16, analog-devices-01:SOIC127P1032X265-16N
- moved TP7 436.8 mm to (47.0, 41.9)
- moved C2 429.4 mm to (22.9, 49.5)
- moved SJ7 424.7 mm to (44.5, 61.0)
- moved SJ8 424.7 mm to (44.5, 55.9)
- moved R16 398.1 mm to (22.9, 47.0), turned to 180 degrees
- moved R15 390.8 mm to (19.1, 47.0)
- moved C1 387.3 mm to (19.1, 49.5), turned to 180 degrees
- moved U1 381.3 mm to (20.3, 53.3)
- moved SJ6 374.4 mm to (44.5, 53.3)
- moved C14 347.2 mm to (38.1, 33.0), turned to 90 degrees
- moved C13 346.9 mm to (40.6, 38.1), turned to 270 degrees
- moved C11 330.4 mm to (40.6, 33.0), turned to 270 degrees
- moved R14 328.3 mm to (38.1, 38.1), turned to 270 degrees
- moved C10 310.9 mm to (35.6, 33.0), turned to 90 degrees
- moved C9 299.2 mm to (35.6, 38.1), turned to 270 degrees
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Connections:
- removed net +VS: U9.8
- removed net -VS: U9.4
- new net GND: C19.1, C21.1, C25.1, C3.1, C4.1, U6.8, U6.9
- new net N$1: U$1.4
- new net N$10: U$1.16
- new net N$12: U$1.18
- new net N$13: U$1.20
- new net N$15: U$1.22
- new net N$2: U$1.6
- new net N$20: U$1.24
- new net N$24: U$1.26
- new net N$26: U$1.28
- new net N$3: R24.2, R28.1, U6.14
- new net N$32: U$1.30
- new net N$33: U$1.40
- new net N$35: U$1.42
- new net N$36: U$1.44
- new net N$37: U$1.46
- new net N$38: U$1.2
- new net N$39: U$1.45
- new net N$40: U$1.43
- new net N$41: U$1.41
- new net N$42: U$1.39
- new net N$43: U$1.29
- new net N$44: U$1.27
- new net N$45: U$1.25
- new net N$46: U$1.23
- new net N$47: U$1.21
- new net N$48: U$1.17
- new net N$49: U$1.15
- new net N$5: U$1.12
- new net N$50: U$1.5
- new net N$51: U$1.75
- new net N$52: R23.2, R27.1, U6.12
- new net N$53: C21.2, R17.1, R18.2, U3.5
- new net N$54: C4.2, R19.1, R20.2, U3.3
- new net N$55: R22.2, R26.1, U6.5
- new net N$56: R21.2, R25.1, U6.3
- new net N$57: C3.2, R20.1
- new net N$58: C20.1
- new net N$59: R18.1
- new net N$6: U$1.14
- new net VBIAS_DOWN: C25.2, U3.6, U3.7, U6.11, U6.15, U6.2, U6.6
- new net VBIAS_UP: C19.2, R29.2, R38.2, R39.1, R39.2, R40.1, R40.2, R41.1, R41.2, R42.1, R42.2, R43.2, R44.2, U10.2, U10.6, U11.2, U11.6, U3.1, U3.2
- net ADC_A: now also U10.3
- net ADC_B: now also U10.5
- net ADC_C: now also U11.3
- net ADC_D: now also U11.5
- net AGND: no longer U$1.2
- net VDD: now also R19.2, U10.8, U11.8, U3.8, U6.4
- net VSS: now also R17.2, U10.4, U11.4, U3.4, U6.13
- net _ADC_A: now also R38.1, U10.1
- net _ADC_B: now also R29.1, U10.7
- net _ADC_C: now also R43.1, U11.1
- net _ADC_D: now also R44.1, U11.7
- net _DAC_A: now also R21.1, R28.2, U6.16
- net _DAC_B: now also R24.1, R25.2, U6.1
- net _DAC_C: now also R23.1, R26.2, U6.7
- net _DAC_D: now also R22.1, R27.2, U6.10
