File: pcb/pcb/boneclamp_rB.sch (EAGLE design)
At the start: 72 parts, among them IC1 24C, U1 AD8032ARZ-REEL7, U2 LT1964ES5-5TRMPBF, U4 TLV70245DBVT, U7 AD7682BCPZ, U8 TPS63700DRCT, U9 ADA4841-2YRZ

Commit message: Added voltage biasing
Parts:
- removed U9: ADA4841-2YRZ, analog-devices-01:ADA4841-2YRZ
- added C19, C20, C21, C25, C3, C4: (no value), resistor:C-EU025-025X050
- added R17: 6.66k, resistor:R-US_0204/2V
- added R18, R20: 10k, resistor:R-US_0204/2V
- added R19: 6.937k, resistor:R-US_0204/2V
- added R21, R22, R23, R24, R25, R26, R27, R28: (no value), resistor:R-US_0204/2V
- added R29, R38, R43, R44: 0.1k, rcl:R-US_R0805
- added R39, R40, R41, R42: 10k, rcl:R-US_R0805
- added U10, U11, U3: ADA4841-2YRZ, analog-devices-01:ADA4841-2YRZ
- added U6: AD713JRZ-16, analog-devices-01:AD713JRZ-16
Connections:
- new net GND: C19.1, C21.1, C25.1, C3.1, C4.1, U6.NC, U6.NC_2
- new net N$1: U$1.GPIO1_7
- new net N$10: U$1.GPIO1_14
- new net N$12: U$1.GPIO2_1
- new net N$13: U$1.GPIO1_31
- new net N$15: U$1.GPIO1_5
- new net N$2: U$1.GPIO1_3
- new net N$20: U$1.GPIO1_1
- new net N$24: U$1.GPIO1_29
- new net N$26: U$1.GPIO2_24
- new net N$3: R24.2, R28.1, U6.+IN
- new net N$32: U$1.GPIO2_25
- new net N$33: U$1.GPIO2_13
- new net N$35: U$1.GPIO2_11
- new net N$36: U$1.GPIO2_9
- new net N$37: U$1.GPIO2_7
- new net N$38: U$1.GND@8
- new net N$39: U$1.GPIO2_6
- new net N$40: U$1.GPIO2_8
- new net N$41: U$1.GPIO2_10
- new net N$42: U$1.GPIO2_12
- new net N$43: U$1.GPIO2_23
- new net N$44: U$1.GPIO2_22
- new net N$45: U$1.GPIO1_0
- new net N$46: U$1.GPIO1_4
- new net N$47: U$1.GPIO1_30
- new net N$48: U$1.GPIO0_27
- new net N$49: U$1.GPIO1_15
- new net N$5: U$1.GPIO1_12
- new net N$50: U$1.GPIO1_2
- new net N$51: U$1.SPI1_DO
- new net N$52: R23.2, R27.1, U6.+IN_4
- new net N$53: C21.2, R17.1, R18.2, U3.+IN2
- new net N$54: C4.2, R19.1, R20.2, U3.+IN1
- new net N$55: R22.2, R26.1, U6.+IN_3
- new net N$56: R21.2, R25.1, U6.+IN_2
- new net N$57: C3.2, R20.1
- new net N$58: C20.1
- new net N$59: R18.1
- new net N$6: U$1.GPIO0_26
- new net VBIAS_DOWN: C25.2, U3.-IN2, U3.OUT2, U6.-IN, U6.-IN_2, U6.-IN_3, U6.-IN_4
- new net VBIAS_UP: C19.2, R29.2, R38.2, R39.1, R39.2, R40.1, R40.2, R41.1, R41.2, R42.1, R42.2, R43.2, R44.2, U10.-IN1, U10.-IN2, U11.-IN1, U11.-IN2, U3.-IN1, U3.OUT1
- net ADC_A: now also U10.+IN1
- net ADC_B: now also U10.+IN2
- net ADC_C: now also U11.+IN1
- net ADC_D: now also U11.+IN2
- net VDD: now also R19.2, U10.+VS, U11.+VS, U3.+VS, U6.+VS
- net VSS: now also R17.2, U10.-VS, U11.-VS, U3.-VS, U6.-VS
- net _ADC_A: now also R38.1, U10.OUT1
- net _ADC_B: now also R29.1, U10.OUT2
- net _ADC_C: now also R43.1, U11.OUT1
- net _ADC_D: now also R44.1, U11.OUT2
- net _DAC_A: now also R21.1, R28.2, U6.OUT
- net _DAC_B: now also R24.1, R25.2, U6.OUT_2
- net _DAC_C: now also R23.1, R26.2, U6.OUT_3
- net _DAC_D: now also R22.1, R27.2, U6.OUT_4
